File: hardware/hardware-jst/hardware.kicad_sch (KiCad schematic)
At the start: 81 parts, among them J2 Barrel_Jack, M1 Stepper_Motor_unipolar_5pin, M10 Stepper_Motor_unipolar_5pin, M11 Stepper_Motor_unipolar_5pin, M12 Stepper_Motor_unipolar_5pin, M13 Stepper_Motor_unipolar_5pin, M14 Stepper_Motor_unipolar_5pin, M2 Stepper_Motor_unipolar_5pin, M3 Stepper_Motor_unipolar_5pin, M4 Stepper_Motor_unipolar_5pin, M5 Stepper_Motor_unipolar_5pin, M6 Stepper_Motor_unipolar_5pin, M7 Stepper_Motor_unipolar_5pin, M8 Stepper_Motor_unipolar_5pin, M9 Stepper_Motor_unipolar_5pin, SW1 SW_Push_SPDT, SW10 SW_Push_SPDT, SW11 SW_Push_SPDT, SW12 SW_Push_SPDT, SW13 SW_Push_SPDT, SW14 SW_Push_SPDT, SW15 SW_Push_SPDT, SW16 SW_Push_SPDT, SW2 SW_Push_SPDT, SW3 SW_Push_SPDT, SW4 SW_Push_SPDT, SW5 SW_Push_SPDT, SW6 SW_Push_SPDT, SW7 SW_Push_SPDT, SW8 SW_Push_SPDT, SW9 SW_Push_SPDT, U1 WeMos_D1_mini, U10 ULN2003A, U11 ULN2003A, U12 ULN2003A, U13 ULN2003A, U14 ULN2003A, U15 ULN2003A, U16 ULN2003A, U17 ULN2003A, U2 CD4051B, U3 CD4051B, U4 ULN2003A, U5 ULN2003A, U6 ULN2003A, U7 ULN2003A, U8 ULN2003A, U9 ULN2003A

Commit message: partial jst conversion of pcb
Parts:
- C1, C10, C11, C12, C13, C14, C2, C3, C4, C5, C6, C7, C8, C9: footprint Capacitor_SMD:C_0805_2012Metric -> Capacitor_SMD:C_0402_1005Metric; LCSC PN C157608 -> C1545
- M1, M10, M11, M12, M13, M14, M2, M3, M4, M7, M8, M9: footprint Connector_Audio:HOOYA-PJ-3505A_C19190915-Jack_3.5mm_PJ31060-I_Horizontal -> Connector_JST:JST_XH_B5B-XH-A_1x05_P2.50mm_Vertical; LCSC PN C19190915 -> (none); LSCS PN (none) -> C157991
- M5, M6: footprint Connector_Audio:HOOYA-PJ-3505A_C19190915-Jack_3.5mm_PJ31060-I_Horizontal -> Connector_JST:JST_XH_B5B-XH-A_1x05_P2.50mm_Vertical; LSCS PN C19190915 -> C157991
Connections:
- net +5V: now also M1.5, M10.5, M11.5, M12.5, M13.5, M14.5, M2.5, M3.5, M4.5, M5.5, M6.5, M7.5, M8.5, M9.5; no longer M1.1, M10.1, M11.1, M12.1, M13.1, M14.1, M2.1, M3.1, M4.1, M5.1, M6.1, M7.1, M8.1, M9.1
- net BLUE1: now also M1.1; no longer M1.5
- net BLUE10: now also M10.1; no longer M10.5
- net BLUE11: now also M11.1; no longer M11.5
- net BLUE12: now also M12.1; no longer M12.5
- net BLUE13: now also M13.1; no longer M13.5
- net BLUE14: now also M14.1; no longer M14.5
- net BLUE2: now also M2.1; no longer M2.5
- net BLUE3: now also M3.1; no longer M3.5
- net BLUE4: now also M4.1; no longer M4.5
- net BLUE5: now also M5.1; no longer M5.5
- net BLUE6: now also M6.1; no longer M6.5
- net BLUE7: now also M7.1; no longer M7.5
- net BLUE8: now also M8.1; no longer M8.5
- net BLUE9: now also M9.1; no longer M9.5
- net ORANGE1: now also M1.4; no longer M1.2
- net ORANGE10: now also M10.4; no longer M10.2
- net ORANGE11: now also M11.4; no longer M11.2
- net ORANGE12: now also M12.4; no longer M12.2
- net ORANGE13: now also M13.4; no longer M13.2
- net ORANGE14: now also M14.4; no longer M14.2
- net ORANGE2: now also M2.4; no longer M2.2
- net ORANGE3: now also M3.4; no longer M3.2
- net ORANGE4: now also M4.4; no longer M4.2
- net ORANGE5: now also M5.4; no longer M5.2
- net ORANGE6: now also M6.4; no longer M6.2
- net ORANGE7: now also M7.4; no longer M7.2
- net ORANGE8: now also M8.4; no longer M8.2
- net ORANGE9: now also M9.4; no longer M9.2
- net PINK1: now also M1.2; no longer M1.3 (-)
- net PINK10: now also M10.2; no longer M10.3 (-)
- net PINK11: now also M11.2; no longer M11.3 (-)
- net PINK12: now also M12.2; no longer M12.3 (-)
- net PINK13: now also M13.2; no longer M13.3 (-)
- net PINK14: now also M14.2; no longer M14.3 (-)
- net PINK2: now also M2.2; no longer M2.3 (-)
- net PINK3: now also M3.2; no longer M3.3 (-)
- net PINK4: now also M4.2; no longer M4.3 (-)
- net PINK5: now also M5.2; no longer M5.3 (-)
- net PINK6: now also M6.2; no longer M6.3 (-)
- net PINK7: now also M7.2; no longer M7.3 (-)
- net PINK8: now also M8.2; no longer M8.3 (-)
- net PINK9: now also M9.2; no longer M9.3 (-)
- net YELLOW1: now also M1.3 (-); no longer M1.4
- net YELLOW10: now also M10.3 (-); no longer M10.4
- net YELLOW11: now also M11.3 (-); no longer M11.4
- net YELLOW12: now also M12.3 (-); no longer M12.4
- net YELLOW13: now also M13.3 (-); no longer M13.4
- net YELLOW14: now also M14.3 (-); no longer M14.4
- net YELLOW2: now also M2.3 (-); no longer M2.4
- net YELLOW3: now also M3.3 (-); no longer M3.4
- net YELLOW4: now also M4.3 (-); no longer M4.4
- net YELLOW5: now also M5.3 (-); no longer M5.4
- net YELLOW6: now also M6.3 (-); no longer M6.4
- net YELLOW7: now also M7.3 (-); no longer M7.4
- net YELLOW8: now also M8.3 (-); no longer M8.4
- net YELLOW9: now also M9.3 (-); no longer M9.4
Other:
- note added: "CHOOSE YOUR COMPONENTS FROM HERE: https://jlcpcb.com/parts/2nd/Capacitors/Multilayer_Ceramic_Capacitors_MLCC_SMD_SMT_33?spm=search&searchTxt=10pf%20 the jlcpcb parts lib and not lcsc!!"
- moved on the sheet: C10, C11, C12, C13, C14, C5, C6, C7, C8, C9, U10, U11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
